Commit message: commit

File: vehicle/aps_vehicle_launch/aps_vehicle_description/urdf/vehicle.xacro (robot description, xacro)
@@ -6,7 +6,8 @@
   <link name="base_link">
     <visual>
-      <origin xyz="${vehicle_info['/**']['ros__parameters']['wheel_base']/2.0} 0 0" rpy="${pi/2.0} 0 ${pi}"/>
+      <!-- <origin xyz="${vehicle_info['/**']['ros__parameters']['wheel_base']/2.0} 0 0" rpy="${pi/2.0} 0 ${pi}"/> -->
+      <origin xyz="0.3 0 0.1" rpy="0.0 0 ${pi/2*3}"/>
       <geometry>
-        <mesh filename="package://aps_vehicle_description/mesh/lexus.dae" scale="1 1 1"/>
+        <mesh filename="package://aps_vehicle_description/mesh/aps2.dae" scale="1 1 1"/>
       </geometry>
     </visual>

Commit message: commit

File: vehicle/aps_vehicle_launch/aps_vehicle_description/urdf/vehicle.xacro (robot description, xacro)
@@ -7,5 +7,5 @@
     <visual>
       <!-- <origin xyz="${vehicle_info['/**']['ros__parameters']['wheel_base']/2.0} 0 0" rpy="${pi/2.0} 0 ${pi}"/> -->
-      <origin xyz="0.3 0 0.1" rpy="0.0 0 ${pi/2*3}"/>
+      <origin xyz="0.2 0 0.1" rpy="0.0 0 ${pi/2*3}"/>
       <geometry>
         <mesh filename="package://aps_vehicle_description/mesh/aps2.dae" scale="1 1 1"/>
