Commit message: add point con

File: sensor_kit/sample_sensor_kit_launch/aps_sensor_kit_description/urdf/sensor_kit.xacro (robot description, xacro)
@@ -4,6 +4,7 @@
     <xacro:include filename="$(find velodyne_description)/urdf/VLP-16.urdf.xacro"/>
     <xacro:include filename="$(find vls_description)/urdf/VLS-128.urdf.xacro"/>
-    <xacro:include filename="$(find camera_description)/urdf/monocular_camera.xacro"/>
     <xacro:include filename="$(find imu_description)/urdf/imu.xacro"/>
+    <xacro:include filename="$(find olei_description)/urdf/LR1BS5.urdf.xacro"/>
+    <xacro:include filename="$(find robosense_description)/urdf/robosense.urdf.xacro"/>
     <xacro:arg name="gpu" default="false"/>
     <xacro:arg name="config_dir" default="$(find sample_sensor_kit_description)/config"/>
@@ -20,5 +21,5 @@
     <xacro:property name="calibration" value="${xacro.load_yaml('$(arg config_dir)/sensor_kit_calibration.yaml')}"/>
     <!-- lidar -->
-    <xacro:VLP-16 parent="sensor_kit_base_link" name="rslidar" topic="/points_raw" hz="10" samples="220" gpu="$(arg gpu)">
+    <xacro:Robosense parent="sensor_kit_base_link" name="rslidar" topic="/points_raw" hz="10" samples="220" gpu="$(arg gpu)">
       <origin
         xyz="${calibration['sensor_kit_base_link']['rslidar']['x']}
@@ -29,159 +30,25 @@
              ${calibration['sensor_kit_base_link']['rslidar']['yaw']}"
       />
-    </xacro:VLP-16>
-    <!-- <xacro:VLP-16 parent="sensor_kit_base_link" name="velodyne_left" topic="/points_raw" hz="10" samples="220" gpu="$(arg gpu)">
+    </xacro:Robosense>
+     <xacro:LR1BS5 parent="sensor_kit_base_link" name="olei_front" topic="/cloud_front" hz="10"  gpu="$(arg gpu)">
       <origin
-        xyz="${calibration['sensor_kit_base_link']['velodyne_left_base_link']['x']}
-             ${calibration['sensor_kit_base_link']['velodyne_left_base_link']['y']}
-             ${calibration['sensor_kit_base_link']['velodyne_left_base_link']['z']}"
-        rpy="${calibration['sensor_kit_base_link']['velodyne_left_base_link']['roll']}
-             ${calibration['sensor_kit_base_link']['velodyne_left_base_link']['pitch']}
-             ${calibration['sensor_kit_base_link']['velodyne_left_base_link']['yaw']}"
+        xyz="${calibration['sensor_kit_base_link']['olei_front_base_link']['x']}
+             ${calibration['sensor_kit_base_link']['olei_front_base_link']['y']}
+             ${calibration['sensor_kit_base_link']['olei_front_base_link']['z']}"
+        rpy="${calibration['sensor_kit_base_link']['olei_front_base_link']['roll']}
+             ${calibration['sensor_kit_base_link']['olei_front_base_link']['pitch']}
+             ${calibration['sensor_kit_base_link']['olei_front_base_link']['yaw']}"
       />
-    </xacro:VLP-16>
-    <xacro:VLP-16 parent="sensor_kit_base_link" name="velodyne_right" topic="/points_raw" hz="10" samples="220" gpu="$(arg gpu)">
+    </xacro:LR1BS5>
+    <xacro:LR1BS5 parent="sensor_kit_base_link" name="olei_back" topic="/cloud_back" hz="10"  gpu="$(arg gpu)">
       <origin
-        xyz="${calibration['sensor_kit_base_link']['velodyne_right_base_link']['x']}
-             ${calibration['sensor_kit_base_link']['velodyne_right_base_link']['y']}
-             ${calibration['sensor_kit_base_link']['velodyne_right_base_link']['z']}"
-        rpy="${calibration['sensor_kit_base_link']['velodyne_right_base_link']['roll']}
-             ${calibration['sensor_kit_base_link']['velodyne_right_base_link']['pitch']}
-             ${calibration['sensor_kit_base_link']['velodyne_right_base_link']['yaw']}"
+        xyz="${calibration['sensor_kit_base_link']['olei_back_base_link']['x']}
+             ${calibration['sensor_kit_base_link']['olei_back_base_link']['y']}
+             ${calibration['sensor_kit_base_link']['olei_back_base_link']['z']}"
+        rpy="${calibration['sensor_kit_base_link']['olei_back_base_link']['roll']}
+             ${calibration['sensor_kit_base_link']['olei_back_base_link']['pitch']}
+             ${calibration['sensor_kit_base_link']['olei_back_base_link']['yaw']}"
       />
-    </xacro:VLP-16> -->
-    <!-- camera -->
-    <!-- <xacro:monocular_camera_macro
-      name="traffic_light_right_camera/camera"
-      parent="sensor_kit_base_link"
-      namespace=""
-      x="${calibration['sensor_kit_base_link']['traffic_light_right_camera/camera_link']['x']}"
-      y="${calibration['sensor_kit_base_link']['traffic_light_right_camera/camera_link']['y']}"
-      z="${calibration['sensor_kit_base_link']['traffic_light_right_camera/camera_link']['z']}"
-      roll="${calibration['sensor_kit_base_link']['traffic_light_right_camera/camera_link']['roll']}"
-      pitch="${calibration['sensor_kit_base_link']['traffic_light_right_camera/camera_link']['pitch']}"
-      yaw="${calibration['sensor_kit_base_link']['traffic_light_right_camera/camera_link']['yaw']}"
-      fps="30"
-      width="800"
-      height="400"
-      fov="1.3"
-    />
-    <xacro:monocular_camera_macro
-      name="traffic_light_left_camera/camera"
-      parent="sensor_kit_base_link"
-      namespace=""
-      x="${calibration['sensor_kit_base_link']['traffic_light_left_camera/camera_link']['x']}"
-      y="${calibration['sensor_kit_base_link']['traffic_light_left_camera/camera_link']['y']}"
-      z="${calibration['sensor_kit_base_link']['traffic_light_left_camera/camera_link']['z']}"
-      roll="${calibration['sensor_kit_base_link']['traffic_light_left_camera/camera_link']['roll']}"
-      pitch="${calibration['sensor_kit_base_link']['traffic_light_left_camera/camera_link']['pitch']}"
-      yaw="${calibration['sensor_kit_base_link']['traffic_light_left_camera/camera_link']['yaw']}"
-      fps="30"
-      width="800"
-      height="400"
-      fov="1.3"
-    />
-    <xacro:monocular_camera_macro
-      name="camera0/camera"
-      parent="sensor_kit_base_link"
-      namespace=""
-      x="${calibration['sensor_kit_base_link']['camera0/camera_link']['x']}"
-      y="${calibration['sensor_kit_base_link']['camera0/camera_link']['y']}"
-      z="${calibration['sensor_kit_base_link']['camera0/camera_link']['z']}"
-      roll="${calibration['sensor_kit_base_link']['camera0/camera_link']['roll']}"
-      pitch="${calibration['sensor_kit_base_link']['camera0/camera_link']['pitch']}"
-      yaw="${calibration['sensor_kit_base_link']['camera0/camera_link']['yaw']}"
-      fps="30"
-      width="800"
-      height="400"
-      fov="1.3"
-    />
-    <xacro:monocular_camera_macro
-      name="camera1/camera"
-      parent="sensor_kit_base_link"
-      namespace=""
-      x="${calibration['sensor_kit_base_link']['camera1/camera_link']['x']}"
-      y="${calibration['sensor_kit_base_link']['camera1/camera_link']['y']}"
-      z="${calibration['sensor_kit_base_link']['camera1/camera_link']['z']}"
-      roll="${calibration['sensor_kit_base_link']['camera1/camera_link']['roll']}"
-      pitch="${calibration['sensor_kit_base_link']['camera1/camera_link']['pitch']}"
-      yaw="${calibration['sensor_kit_base_link']['camera1/camera_link']['yaw']}"
-      fps="30"
-      width="800"
-      height="400"
-      fov="1.3"
-    />
-    <xacro:monocular_camera_macro
-      name="camera2/camera"
-      parent="sensor_kit_base_link"
-      namespace=""
-      x="${calibration['sensor_kit_base_link']['camera2/camera_link']['x']}"
-      y="${calibration['sensor_kit_base_link']['camera2/camera_link']['y']}"
-      z="${calibration['sensor_kit_base_link']['camera2/camera_link']['z']}"
-      roll="${calibration['sensor_kit_base_link']['camera2/camera_link']['roll']}"
-      pitch="${calibration['sensor_kit_base_link']['camera2/camera_link']['pitch']}"
-      yaw="${calibration['sensor_kit_base_link']['camera2/camera_link']['yaw']}"
-      fps="30"
-      width="800"
-      height="400"
-      fov="1.3"
-    />
-    <xacro:monocular_camera_macro
-      name="camera3/camera"
-      parent="sensor_kit_base_link"
-      namespace=""
-      x="${calibration['sensor_kit_base_link']['camera3/camera_link']['x']}"
-      y="${calibration['sensor_kit_base_link']['camera3/camera_link']['y']}"
-      z="${calibration['sensor_kit_base_link']['camera3/camera_link']['z']}"
-      roll="${calibration['sensor_kit_base_link']['camera3/camera_link']['roll']}"
-      pitch="${calibration['sensor_kit_base_link']['camera3/camera_link']['pitch']}"
-      yaw="${calibration['sensor_kit_base_link']['camera3/camera_link']['yaw']}"
-      fps="30"
-      width="800"
-      height="400"
-      fov="1.3"
-    />
-    <xacro:monocular_camera_macro
-      name="camera4/camera"
-      parent="sensor_kit_base_link"
-      namespace=""
-      x="${calibration['sensor_kit_base_link']['camera4/camera_link']['x']}"
-      y="${calibration['sensor_kit_base_link']['camera4/camera_link']['y']}"
-      z="${calibration['sensor_kit_base_link']['camera4/camera_link']['z']}"
-      roll="${calibration['sensor_kit_base_link']['camera4/camera_link']['roll']}"
-      pitch="${calibration['sensor_kit_base_link']['camera4/camera_link']['pitch']}"
-      yaw="${calibration['sensor_kit_base_link']['camera4/camera_link']['yaw']}"
-      fps="30"
-      width="800"
-      height="400"
-      fov="1.3"
-    />
-    <xacro:monocular_camera_macro
-      name="camera5/camera"
-      parent="sensor_kit_base_link"
-      namespace=""
-      x="${calibration['sensor_kit_base_link']['camera5/camera_link']['x']}"
-      y="${calibration['sensor_kit_base_link']['camera5/camera_link']['y']}"
-      z="${calibration['sensor_kit_base_link']['camera5/camera_link']['z']}"
-      roll="${calibration['sensor_kit_base_link']['camera5/camera_link']['roll']}"
-      pitch="${calibration['sensor_kit_base_link']['camera5/camera_link']['pitch']}"
-      yaw="${calibration['sensor_kit_base_link']['camera5/camera_link']['yaw']}"
-      fps="30"
-      width="800"
-      height="400"
-      fov="1.3"
-    /> -->
-    <!-- gnss -->
-    <!-- <xacro:imu_macro
-      name="gnss"
-      parent="sensor_kit_base_link"
-      namespace=""
-      x="${calibration['sensor_kit_base_link']['gnss_link']['x']}"
-      y="${calibration['sensor_kit_base_link']['gnss_link']['y']}"
-      z="${calibration['sensor_kit_base_link']['gnss_link']['z']}"
-      roll="${calibration['sensor_kit_base_link']['gnss_link']['roll']}"
-      pitch="${calibration['sensor_kit_base_link']['gnss_link']['pitch']}"
-      yaw="${calibration['sensor_kit_base_link']['gnss_link']['yaw']}"
-      fps="100"
-    /> -->
+    </xacro:LR1BS5>
     <!-- imu -->
     <xacro:imu_macro

File: vehicle/aps_vehicle_launch/aps_vehicle_description/urdf/vehicle.xacro (robot description, xacro)
@@ -7,5 +7,5 @@
     <visual>
       <!-- <origin xyz="${vehicle_info['/**']['ros__parameters']['wheel_base']/2.0} 0 0" rpy="${pi/2.0} 0 ${pi}"/> -->
-      <origin xyz="0.2 0 0.1" rpy="0.0 0 ${pi/2*3}"/>
+      <origin xyz="0.2 0 0.11" rpy="0.0 0 ${pi/2*3}"/>
       <geometry>
         <mesh filename="package://aps_vehicle_description/mesh/aps2.dae" scale="1 1 1"/>
